File: reward_port/pcb/controller.brd (EAGLE design)
At the start: 76.2 x 38.1 mm, 18 parts, among them J2 COMPUTER-PERIPHERAL-POWERRA

Commit message: controller routing
Parts:
- moved R2 11.1 mm to (22.2, 25.8), turned to 270 degrees
- moved R3 10.8 mm to (32.9, 25.7), turned to 270 degrees
- moved R4 7.88 mm to (-28.7, 44.5), turned to 90 degrees
- moved R5 3.59 mm to (-28.7, 40.6), turned to 270 degrees
- moved R8 1.14 mm to (17.8, 29.2)
Routing:
- net 12V: track 0.00 -> 56.2 mm, vias 0 -> 1
- net I2C_SCL: track 0.00 -> 42.1 mm
- net I2C_SDA: track 0.00 -> 42.1 mm
- net 3.3V: track 0.00 -> 32.1 mm
- net VDD: track 1.80 -> 33.2 mm
- net GND: track 0.00 -> 28.4 mm
- net N$11: track 0.00 -> 25.8 mm
- net N$9: track 0.00 -> 22.1 mm
- net N$8: track 0.00 -> 18.5 mm
- net N$17: track 0.00 -> 17.8 mm
- net N$12: track 0.00 -> 15.5 mm
- net N$13: track 0.00 -> 15.0 mm
- net N$6: track 0.00 -> 14.9 mm
- net VDD5-REG: track 0.00 -> 9.92 mm
- net VDD5-IN: track 0.00 -> 7.10 mm
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